File: cookpad-pad.kicad_pcb (KiCad board)
At the start: 2 copper layers, 79.4 x 47.6 mm, 21 parts, among them SW1 SW_Push

Commit message: Update PCB
Parts:
- removed the ? at (111.9, 96.8)
- added J1: LED, Cookpad-Pad:LED_Strip, F.Cu at (111.9, 86.5)
- D1, D2, D3, D4, D5, D6: footprint random-keyboard-parts:D_SOD-123-Pretty -> Cookpad-Pad:D3_TH_SMD
- moved D2 5.12 mm to (140.7, 85.3)
- moved D6 4.92 mm to (159.5, 87.6)
- moved D4 4.92 mm to (121.4, 87.6)
- moved D1 4.87 mm to (121.4, 85.3)
- moved D3 4.87 mm to (159.5, 85.3)
- moved D5 4.67 mm to (140.7, 87.6)
- moved U1 1.59 mm to (100.0, 84.9)
- moved SW1 0.48 mm to (100.0, 102.9)
- gave numbers to parts that had none: 1
Connections:
- U1 pad 10: Net-(U1-Pad10) -> (no net)
- U1 pad 11: Net-(U1-Pad11) -> (no net)
- U1 pad 12: Net-(U1-Pad12) -> (no net)
- U1 pad 13: Net-(U1-Pad13) -> (no net)
- U1 pad 14: Net-(U1-Pad14) -> (no net)
- U1 pad 15: Net-(U1-Pad15) -> (no net)
- U1 pad 2: Net-(U1-Pad2) -> (no net)
- U1 pad 24: Net-(U1-Pad24) -> (no net)
- U1 pad 5: Net-(U1-Pad5) -> (no net)
- U1 pad 6: Net-(U1-Pad6) -> (no net)
- U1 pad 7: Net-(U1-Pad7) -> (no net)
- U1 pad 8: Net-(U1-Pad8) -> (no net)
- U1 pad 9: Net-(U1-Pad9) -> (no net)
Routing:
- net VCC: track 15.9 -> 7.17 mm
- net led: track 45.0 -> 38.1 mm
- net GND: track 77.5 -> 82.6 mm
- net row1: track 59.0 -> 62.2 mm
- net col0: track 34.7 -> 37.3 mm
- net row0: track 51.2 -> 53.7 mm
- net Net-(D5-Pad2): track 6.05 -> 7.52 mm
- net Net-(D1-Pad2): track 17.4 -> 16.0 mm
- net Net-(D3-Pad2): track 17.4 -> 16.0 mm
- net col1: track 58.9 -> 57.6 mm
- net col2: track 76.2 -> 75.2 mm
- net reset: track 29.8 -> 28.8 mm
- net Net-(D2-Pad2): track 17.4 -> 16.9 mm
- added copper zone on B.Cu, net GND
- removed copper zone on B.Cu, net (none)
Other:
- board text added: "Cookpad Pad ver. 1.1.0 https://cookpad.jobs"
- board text removed: "Cookpad Pad ver. 1.0.0 https://cookpad.jobs"
